Commit message: add mimic joint gazebo plugin

File: lara_description/urdf/pgc140_macro.xacro (robot description, xacro)
@@ -175,11 +175,32 @@
       </actuator>
   </transmission>
+  <xacro:macro name="mimic_joint_plugin_gazebo" params="name_prefix parent_joint mimic_joint has_pid:=false multiplier:=1.0 offset:=0 sensitiveness:=0.0 max_effort:=1.0 robot_namespace:=''">
+    <gazebo>
+      <plugin name="${name_prefix}mimic_joint_plugin" filename="libroboticsgroup_gazebo_mimic_joint_plugin.so">
+        <joint>${parent_joint}</joint>
+        <mimicJoint>${mimic_joint}</mimicJoint>
+        <xacro:if value="${has_pid}">                     <!-- if set to true, PID parameters from "/gazebo_ros_control/pid_gains/${mimic_joint}" are loaded -->
+          <hasPID />
+        </xacro:if>
+        <multiplier>${multiplier}</multiplier>
+        <offset>${offset}</offset>
+        <sensitiveness>${sensitiveness}</sensitiveness>   <!-- if absolute difference between setpoint and process value is below this threshold, do nothing; 0.0 = disable [rad] -->
+        <maxEffort>${max_effort}</maxEffort>              <!-- only taken into account if has_pid:=true [Nm] -->
+        <xacro:unless value="${robot_namespace == ''}">
+          <robotNamespace>${robot_namespace}</robotNamespace>
+        </xacro:unless>
+      </plugin>
+    </gazebo>
+  </xacro:macro>
+  <xacro:mimic_joint_plugin_gazebo name_prefix="finger2_joint"
+    parent_joint="finger1_joint" mimic_joint="finger2_joint"
+    has_pid="true" multiplier="1.0" max_effort="10.0" />
+<!--
   <gazebo>
-    <!-- Fix mimicking bug -->
     <plugin filename="libroboticsgroup_upatras_gazebo_mimic_joint_plugin.so" name="mimicker">
       <joint>finger1_joint</joint>
       <mimicJoint>finger2_joint</mimicJoint>
     </plugin>
-  </gazebo>
+  </gazebo> -->
   </xacro:macro>
 </robot>
