Commit message: working gazebo

File: lara_description/urdf/aubo_i5_macro.xacro (robot description, xacro)
@@ -88,5 +88,5 @@
     </xacro:macro>
     <!--/////////////////////////////// BASE_LINK ////////////////////////////////////-->
-   <link name="base_link">
+   <link name="aubo_i5_base_link">
     <inertial>
       <origin xyz="-1.4795E-13 0.0015384 0.020951" rpy="0 0 0" />
@@ -134,5 +134,5 @@
   <joint name="shoulder_joint" type="revolute">
     <origin xyz="0 0 0.122" rpy="0 0 3.1416" />
-    <parent link="base_link" />
+    <parent link="aubo_i5_base_link" />
     <child link="shoulder_Link" />
     <axis xyz="0 0 1" />
@@ -294,4 +294,5 @@
        <actuator name="${joint_name}_motor">
          <mechanicalReduction>1</mechanicalReduction>
+         <hardwareInterface>hardware_interface/PositionJointInterface</hardwareInterface>
        </actuator>
      </transmission>
@@ -303,10 +304,4 @@
   <xacro:aubo_arm_transmission joint_name="wrist2_joint"/>
   <xacro:aubo_arm_transmission joint_name="wrist3_joint"/>
-  <!-- ros_control plugin -->
-  <gazebo>
-      <plugin name="gazebo_ros_control" filename="libgazebo_ros_control.so">
-          <robotNamespace>/aubo_i5</robotNamespace>
-      </plugin>
-  </gazebo>
 </xacro:macro>
 </robot>

File: lara_description/urdf/pgc140_macro.xacro (robot description, xacro)
@@ -4,7 +4,7 @@
      For more information, please see http://wiki.ros.org/sw_urdf_exporter -->
 <robot xmlns:xacro="http://ros.org/wiki/xacro">
-  <xacro:macro name="dh_pgc140">
+  <xacro:macro name="pgc140">
   <link
-    name="base_link">
+    name="pgc140_base_link">
     <inertial>
       <origin
@@ -92,5 +92,5 @@
       rpy="0 0 -1.5708" />
     <parent
-      link="base_link" />
+      link="pgc140_base_link" />
     <child
       link="finger1_link" />
@@ -150,5 +150,5 @@
       rpy="0 0 1.5708" />
     <parent
-      link="base_link" />
+      link="pgc140_base_link" />
     <child
       link="finger2_link" />
@@ -162,7 +162,24 @@
     <mimic
       joint="finger1_joint"
-      multiplier="1"
-      offset="0" />
+      multiplier="1.0"
+      offset="0.0" />
   </joint>
+  <transmission name="finger1_trans">
+      <type>transmission_interface/SimpleTransmission</type>
+      <joint name="finger1_joint">
+          <hardwareInterface>hardware_interface/PositionJointInterface</hardwareInterface>
+      </joint>
+      <actuator name="finger1_motor">
+          <mechanicalReduction>1</mechanicalReduction>
+          <hardwareInterface>hardware_interface/PositionJointInterface</hardwareInterface>
+      </actuator>
+  </transmission>
+  <gazebo>
+    <!-- Fix mimicking bug -->
+    <plugin filename="libroboticsgroup_upatras_gazebo_mimic_joint_plugin.so" name="mimicker">
+      <joint>finger1_joint</joint>
+      <mimicJoint>finger2_joint</mimicJoint>
+    </plugin>
+  </gazebo>
   </xacro:macro>
 </robot>

Commit message: change to effortjointinterface, add gazebo box, pick and place script

File: lara_description/urdf/aubo_i5_macro.xacro (robot description, xacro)
@@ -290,9 +290,9 @@
        <joint name="${joint_name}">
          <!--<hardwareInterface>hardware_interface/PositionJointInterface</hardwareInterface>-->
-         <hardwareInterface>hardware_interface/PositionJointInterface</hardwareInterface>
+         <hardwareInterface>hardware_interface/EffortJointInterface</hardwareInterface>
        </joint>
        <actuator name="${joint_name}_motor">
          <mechanicalReduction>1</mechanicalReduction>
-         <hardwareInterface>hardware_interface/PositionJointInterface</hardwareInterface>
+         <hardwareInterface>hardware_interface/EffortJointInterface</hardwareInterface>
        </actuator>
      </transmission>

File: lara_description/urdf/aubo_i5_pgc140.urdf.xacro (robot description, xacro)
@@ -32,8 +32,21 @@
     <parent link="ee_link"/>
     <child link="gripper_tip_link"/>
-    <origin rpy="0 0 0" xyz="0.163 0 0"/>
+    <origin rpy="0 0 0" xyz="0.13345 0 0"/>
+  </joint>
+  <link name="ground">
+      <collision>
+          <origin rpy="0 0 0" xyz="0 0 -0.01"/>
+          <geometry>
+              <box size="5 5 0.02" />
+          </geometry>
+      </collision>
+  </link>
+  <joint name="ground_to_world" type="fixed">
+      <parent link="world"/>
+      <child link="ground"/>
+      <origin xyz="0 0 0" />
   </joint>
   <link name="world" />
-  <joint name="world_joint" type="fixed">
+  <joint name="aubo_to_world" type="fixed">
     <parent link="world" />
     <child link = "aubo_i5_base_link" />

File: lara_description/urdf/pgc140_macro.xacro (robot description, xacro)
@@ -100,5 +100,5 @@
       lower="0"
       upper="0.025"
-      effort="140"
+      effort="1000"
       velocity="1" />
   </joint>
@@ -158,5 +158,5 @@
       lower="0"
       upper="0.025"
-      effort="140"
+      effort="1000"
       velocity="1" />
     <mimic
@@ -168,9 +168,9 @@
       <type>transmission_interface/SimpleTransmission</type>
       <joint name="finger1_joint">
-          <hardwareInterface>hardware_interface/PositionJointInterface</hardwareInterface>
+          <hardwareInterface>hardware_interface/EffortJointInterface</hardwareInterface>
       </joint>
       <actuator name="finger1_motor">
           <mechanicalReduction>1</mechanicalReduction>
-          <hardwareInterface>hardware_interface/PositionJointInterface</hardwareInterface>
+          <hardwareInterface>hardware_interface/EffortJointInterface</hardwareInterface>
       </actuator>
   </transmission>
@@ -195,12 +195,27 @@
   <xacro:mimic_joint_plugin_gazebo name_prefix="finger2_joint"
     parent_joint="finger1_joint" mimic_joint="finger2_joint"
-    has_pid="true" multiplier="1.0" max_effort="10.0" />
-<!--
-  <gazebo>
-    <plugin filename="libroboticsgroup_upatras_gazebo_mimic_joint_plugin.so" name="mimicker">
-      <joint>finger1_joint</joint>
-      <mimicJoint>finger2_joint</mimicJoint>
-    </plugin>
-  </gazebo> -->
+    has_pid="true" multiplier="1.0" max_effort="1000.0" />
   </xacro:macro>
+  <gazebo reference="finger1_link">
+  <material>Gazebo/Red</material>
+    <mu1>1000000.0</mu1>
+    <mu2>1000000.0</mu2>
+    <kp>1000000.0</kp>
+    <kd>100000.0</kd>
+    <minDepth>0.003</minDepth>
+   <maxVel>0</maxVel>
+   <slip1>0</slip1>
+    <slip2>0</slip2>
+  </gazebo>
+  <gazebo reference="finger2_link">
+  <material>Gazebo/Red</material>
+    <mu1>1000000.0</mu1>
+    <mu2>1000000.0</mu2>
+    <kp>1000000.0</kp>
+    <kd>100000.0</kd>
+    <minDepth>0.003</minDepth>
+   <maxVel>0</maxVel>
+   <slip1>0</slip1>
+    <slip2>0</slip2>
+  </gazebo>
 </robot>
