Commit message: pose tracking and gazebo grasp plugin, effort controller gripper

File: lara_description/urdf/lara_base_scene.xacro (robot description, xacro)
@@ -7,5 +7,5 @@
     <origin xyz="0 0 0" rpy="0 0 0" />
   </xacro:aubo_i5>
-  <xacro:dh_ag95_gripper prefix="" parent="ee_link" transmission_hw_interface="hardware_interface/PositionJointInterface" >
+  <xacro:dh_ag95_gripper prefix="" parent="ee_link" transmission_hw_interface="hardware_interface/EffortJointInterface" >
     <origin xyz="0 0 0" rpy="${pi/2}  ${pi} ${pi/2}" />
   </xacro:dh_ag95_gripper>
@@ -16,4 +16,11 @@
     <child link="gripper_tip_link" />
     <origin rpy="0 0 0" xyz="0.2 0 0" />
+  </joint>
+  <!-- Add an additional link to teleop control with Meta Quest 2 controller. Oriented like the Meta Quest 2 controller frame -->
+  <link name="teleop_link" />
+  <joint name="teleop_link_joint" type="fixed">
+    <parent link="gripper_tip_link" />
+    <child link="teleop_link" />
+    <origin rpy="${-pi/2} 0 ${-pi/2}" xyz="0 0 0" />
   </joint>
   <link name="world" />
@@ -35,3 +42,23 @@
     <plugin name="gazebo_ros_control" filename="libgazebo_ros_control.so"></plugin>
   </gazebo>
+  <!-- gazebo grasp plugin -->
+  <gazebo>
+    <plugin name="gazebo_grasp_fix" filename="libgazebo_grasp_fix.so">
+         <arm>
+            <arm_name>aubo_i5_ag95</arm_name>
+            <palm_link>wrist_3_link</palm_link>
+            <gripper_link>left_inner_finger</gripper_link>
+            <gripper_link>right_inner_finger</gripper_link>
+            <gripper_link>left_inner_knuckle</gripper_link>
+            <gripper_link>right_inner_knuckle</gripper_link>
+         </arm>
+        <forces_angle_tolerance>90</forces_angle_tolerance>
+        <update_rate>30</update_rate>
+        <grip_count_threshold>1</grip_count_threshold>
+        <max_grip_count>3</max_grip_count>
+        <release_tolerance>0.004</release_tolerance>
+        <disable_collisions_on_attach>false</disable_collisions_on_attach>
+        <contact_topic>__default_topic__</contact_topic>
+     </plugin>
+ </gazebo>
 </robot>

File: lara_description/urdf/parts/box.urdf (robot description, URDF)
Before this commit: robot red_box, 1 links, 0 joints
Links:
- link base_link: geometry collision box size=0.04 0.04 0.04; visual box size=0.04 0.04 0.04

Commit message: add different objects, workspace, grasping works!

File: lara_description/urdf/lara_base_scene.xacro (robot description, xacro)
@@ -4,10 +4,22 @@
   <xacro:include filename="$(find aubo_description)/urdf/aubo_i5_macro.xacro" />
   <xacro:include filename="$(find dh_ag95_description)/urdf/ag95_macro.xacro" />
-  <xacro:aubo_i5 prefix="" parent="world" hw_interface="hardware_interface/PositionJointInterface" >
+  <xacro:include filename="$(find lara_description)/urdf/workspace/lara_workspace_macro.xacro" />
+  <xacro:include filename="$(find realsense2_description)/urdf/_d435.urdf.xacro" />
+  <xacro:aubo_i5 prefix="" parent="arm_mount_1" hw_interface="hardware_interface/PositionJointInterface">
     <origin xyz="0 0 0" rpy="0 0 0" />
   </xacro:aubo_i5>
-  <xacro:dh_ag95_gripper prefix="" parent="ee_link" transmission_hw_interface="hardware_interface/EffortJointInterface" >
+  <xacro:dh_ag95_gripper prefix="" parent="ee_link"
+    transmission_hw_interface="hardware_interface/PositionJointInterface">
     <origin xyz="0 0 0" rpy="${pi/2}  ${pi} ${pi/2}" />
   </xacro:dh_ag95_gripper>
+  <xacro:workspace parent="world" arm_mount_spacing="0.4">
+    <origin xyz="0 0 0" rpy="0 0 0" />
+  </xacro:workspace>
+  <!-- <sensor_d435 parent="world" name="camera1" publish_pointcloud="false" topics_ns="camera1">
+    <origin xyz=".75 -0.4 1.5" rpy="0 ${pi/4} ${pi}"/>
+  </sensor_d435>
+  <sensor_d435 parent="world" name="camera2" publish_pointcloud="false" topics_ns="camera2">
+    <origin xyz="0 1 1.2" rpy="0 0 ${-pi/2}"/>
+  </sensor_d435> -->
   <!-- Add an additional link to plan with. Oriented like the aubo_i5 ee_link frame. -->
   <link name="gripper_tip_link" />
@@ -17,5 +29,6 @@
     <origin rpy="0 0 0" xyz="0.2 0 0" />
   </joint>
-  <!-- Add an additional link to teleop control with Meta Quest 2 controller. Oriented like the Meta Quest 2 controller frame -->
+  <!-- Add an additional link to teleop control with Meta Quest 2 controller. Oriented like the Meta
+  Quest 2 controller frame -->
   <link name="teleop_link" />
   <joint name="teleop_link_joint" type="fixed">
@@ -24,18 +37,13 @@
     <origin rpy="${-pi/2} 0 ${-pi/2}" xyz="0 0 0" />
   </joint>
+  <!-- Add an additional frame to plan with. Oriented like world frame. -->
+  <link name="manipulation_frame" />
+  <joint name="manipulation_frame_joint" type="fixed">
+    <parent link="aubo_i5_base_link" />
+    <child link="manipulation_frame" />
+    <origin rpy="0 0 0" xyz="0 0 ${-0.045-0.0225}" />
+  </joint>
+  <!-- world link for gazebo -->
   <link name="world" />
-  <link name="ground">
-    <collision>
-      <origin rpy="0 0 0" xyz="0 0 -0.01" />
-      <geometry>
-        <box size="5 5 0.02" />
-      </geometry>
-    </collision>
-  </link>
-  <joint name="ground_to_world" type="fixed">
-    <parent link="world" />
-    <child link="ground" />
-    <origin xyz="0 0 0" />
-  </joint>
   <!-- ros_control plugin -->
   <gazebo>
@@ -43,22 +51,22 @@
   </gazebo>
   <!-- gazebo grasp plugin -->
-  <gazebo>
+  <!-- <gazebo>
     <plugin name="gazebo_grasp_fix" filename="libgazebo_grasp_fix.so">
-         <arm>
-            <arm_name>aubo_i5_ag95</arm_name>
-            <palm_link>wrist_3_link</palm_link>
-            <gripper_link>left_inner_finger</gripper_link>
-            <gripper_link>right_inner_finger</gripper_link>
-            <gripper_link>left_inner_knuckle</gripper_link>
-            <gripper_link>right_inner_knuckle</gripper_link>
-         </arm>
-        <forces_angle_tolerance>90</forces_angle_tolerance>
-        <update_rate>30</update_rate>
-        <grip_count_threshold>1</grip_count_threshold>
-        <max_grip_count>3</max_grip_count>
-        <release_tolerance>0.004</release_tolerance>
-        <disable_collisions_on_attach>false</disable_collisions_on_attach>
-        <contact_topic>__default_topic__</contact_topic>
-     </plugin>
- </gazebo>
+      <arm>
+        <arm_name>aubo_i5_ag95</arm_name>
+        <palm_link>wrist_3_link</palm_link>
+        <gripper_link>left_finger</gripper_link>
+        <gripper_link>right_finger</gripper_link>
+        <gripper_link>left_inner_knuckle</gripper_link>
+        <gripper_link>right_inner_knuckle</gripper_link>
+      </arm>
+      <forces_angle_tolerance>90</forces_angle_tolerance>
+      <update_rate>30</update_rate>
+      <grip_count_threshold>1</grip_count_threshold>
+      <max_grip_count>3</max_grip_count>
+      <release_tolerance>0.004</release_tolerance>
+      <disable_collisions_on_attach>false</disable_collisions_on_attach>
+      <contact_topic>__default_topic__</contact_topic>
+    </plugin>
+  </gazebo> -->
 </robot>

File: lara_description/urdf/parts/cube.urdf (robot description, URDF)
Before this commit: robot red_box, 1 links, 0 joints
Links:
- link base_link: mass 0.13568 -> .006784; geometry collision box size=0.04 0.04 0.04; visual box size=0.04 0.04 0.04

Commit message: update to get working

File: lara_description/urdf/lara_base_scene.xacro (robot description, xacro)
@@ -5,5 +5,5 @@
   <xacro:include filename="$(find dh_ag95_description)/urdf/ag95_macro.xacro" />
   <xacro:include filename="$(find lara_description)/urdf/workspace/lara_workspace_macro.xacro" />
-  <!-- <xacro:include filename="$(find realsense2_description)/urdf/_d435.urdf.xacro" /> -->
+  <xacro:include filename="$(find realsense2_description)/urdf/_d435.urdf.xacro" />
   <xacro:aubo_i5 prefix="" parent="arm_mount_1" hw_interface="hardware_interface/PositionJointInterface">
     <origin xyz="0 0 0" rpy="0 0 0" />
@@ -50,23 +50,3 @@
     <plugin name="gazebo_ros_control" filename="libgazebo_ros_control.so"></plugin>
   </gazebo>
-  <!-- gazebo grasp plugin -->
-  <!-- <gazebo>
-    <plugin name="gazebo_grasp_fix" filename="libgazebo_grasp_fix.so">
-      <arm>
-        <arm_name>aubo_i5_ag95</arm_name>
-        <palm_link>wrist_3_link</palm_link>
-        <gripper_link>left_finger</gripper_link>
-        <gripper_link>right_finger</gripper_link>
-        <gripper_link>left_inner_knuckle</gripper_link>
-        <gripper_link>right_inner_knuckle</gripper_link>
-      </arm>
-      <forces_angle_tolerance>90</forces_angle_tolerance>
-      <update_rate>30</update_rate>
-      <grip_count_threshold>1</grip_count_threshold>
-      <max_grip_count>3</max_grip_count>
-      <release_tolerance>0.004</release_tolerance>
-      <disable_collisions_on_attach>false</disable_collisions_on_attach>
-      <contact_topic>__default_topic__</contact_topic>
-    </plugin>
-  </gazebo> -->
 </robot>

File: lara_moveit_config/config/gazebo_lara_base_scene.urdf (robot description, URDF)
Before this commit: robot lara_base_scene, 26 links, 25 joints
Joints:
- joint elbow_joint: limit lower=-3.04 upper=3.04 effort=150.0 velocity=50 -> lower=-3.04 upper=3.04 effort=150.0 velocity=1
- joint left_finger_joint: limit lower=-0.01 upper=0.94 effort=50.0 velocity=1.0 -> lower=-0.01 upper=0.94 effort=50.0 velocity=2.0
- joint left_inner_knuckle_joint: limit lower=-0.01 upper=0.94 effort=50.0 velocity=1.0 -> lower=-0.01 upper=0.94 effort=50.0 velocity=2.0
- joint left_outer_knuckle_joint: limit lower=0 upper=0.93 effort=50.0 velocity=1.0 -> lower=0 upper=0.93 effort=50.0 velocity=2.0
- joint right_finger_joint: limit lower=-0.01 upper=0.94 effort=50.0 velocity=1.0 -> lower=-0.01 upper=0.94 effort=50.0 velocity=2.0
- joint right_inner_knuckle_joint: limit lower=-0.01 upper=0.94 effort=50.0 velocity=1.0 -> lower=-0.01 upper=0.94 effort=50.0 velocity=2.0
- joint right_outer_knuckle_joint: limit lower=-0.01 upper=0.94 effort=50.0 velocity=1.0 -> lower=-0.01 upper=0.94 effort=50.0 velocity=2.0
- joint shoulder_lift_joint: limit lower=-3.04 upper=3.04 effort=150.0 velocity=50 -> lower=-3.04 upper=3.04 effort=150.0 velocity=1
- joint shoulder_pan_joint: limit lower=-3.04 upper=3.04 effort=150.0 velocity=50 -> lower=-3.04 upper=3.04 effort=150.0 velocity=1
- joint wrist_1_joint: limit lower=-3.04 upper=3.04 effort=28.0 velocity=50 -> lower=-3.04 upper=3.04 effort=28.0 velocity=1
- joint wrist_2_joint: limit lower=-3.04 upper=3.04 effort=28.0 velocity=50 -> lower=-3.04 upper=3.04 effort=28.0 velocity=1
- joint wrist_3_joint: limit lower=-3.04 upper=3.04 effort=28.0 velocity=50 -> lower=-3.04 upper=3.04 effort=28.0 velocity=1

Commit message: added cameras

File: lara_description/urdf/lara_base_scene.xacro (robot description, xacro)
@@ -2,24 +2,33 @@
 <robot xmlns:xacro="http://ros.org/wiki/xacro"
   name="lara_base_scene">
+  <xacro:arg name="cameras" default="false"/>
   <xacro:include filename="$(find aubo_description)/urdf/aubo_i5_macro.xacro" />
   <xacro:include filename="$(find dh_ag95_description)/urdf/ag95_macro.xacro" />
   <xacro:include filename="$(find lara_description)/urdf/workspace/lara_workspace_macro.xacro" />
   <xacro:include filename="$(find realsense2_description)/urdf/_d435.urdf.xacro" />
+  <!-- world link for gazebo -->
+  <link name="world" />
+  <!-- arm -->
   <xacro:aubo_i5 prefix="" parent="arm_mount_1" hw_interface="hardware_interface/PositionJointInterface">
     <origin xyz="0 0 0" rpy="0 0 0" />
   </xacro:aubo_i5>
+  <!-- gripper -->
   <xacro:dh_ag95_gripper prefix="" parent="ee_link"
     transmission_hw_interface="hardware_interface/PositionJointInterface">
     <origin xyz="0 0 0" rpy="${pi/2}  ${pi} ${pi/2}" />
   </xacro:dh_ag95_gripper>
+  <!-- workspace environment -->
   <xacro:workspace parent="world" arm_mount_spacing="0.4">
     <origin xyz="0 0 0" rpy="0 0 0" />
   </xacro:workspace>
-  <!-- <sensor_d435 parent="world" name="camera1" publish_pointcloud="false" topics_ns="camera1">
-    <origin xyz=".75 -0.4 1.5" rpy="0 ${pi/4} ${pi}"/>
-  </sensor_d435>
-  <sensor_d435 parent="world" name="camera2" publish_pointcloud="false" topics_ns="camera2">
-    <origin xyz="0 1 1.2" rpy="0 0 ${-pi/2}"/>
-  </sensor_d435> -->
+  <!-- optional cameras -->
+  <xacro:if value="$(arg cameras)">
+    <xacro:sensor_d435 parent="world" name="camera1" publish_pointcloud="false" topics_ns="camera1">
+      <origin xyz=".75 -0.4 1.5" rpy="0 ${pi/4} ${pi}"/>
+    </xacro:sensor_d435>
+    <xacro:sensor_d435 parent="world" name="camera2" publish_pointcloud="false" topics_ns="camera2">
+      <origin xyz="0 1 1.2" rpy="0 0 ${-pi/2}"/>
+    </xacro:sensor_d435>
+  </xacro:if>
   <!-- Add an additional link to plan with. Oriented like the aubo_i5 ee_link frame. -->
   <link name="gripper_tip_link" />
@@ -44,6 +53,4 @@
     <origin rpy="0 0 0" xyz="0 0 ${-0.045-0.0225}" />
   </joint>
-  <!-- world link for gazebo -->
-  <link name="world" />
   <!-- ros_control plugin -->
   <gazebo>
