Commit message: lara_simulation tools added

File: lara_moveit_config/config/gazebo_lara_base_scene.urdf (robot description, URDF)
Before this commit: robot lara_base_scene, 26 links, 25 joints
Links:
- link ag95_base_link: mass 0.18321316702693136 -> 0.0533567490598
- link ag95_body: mass 2.681074820833332 -> 0.780803250918
Joints:
- joint elbow_joint: limit lower=-3.04 upper=3.04 effort=150 velocity=3.14159265359 -> lower=-3.04 upper=3.04 effort=150.0 velocity=50
- joint left_finger_joint: limit lower=-0.01 upper=0.94 effort=10.0 velocity=1.0 -> lower=-0.01 upper=0.94 effort=50.0 velocity=1.0
- joint left_inner_knuckle_joint: limit lower=-0.01 upper=0.94 effort=10.0 velocity=1.0 -> lower=-0.01 upper=0.94 effort=50.0 velocity=1.0
- joint left_outer_knuckle_joint: limit lower=0 upper=0.93 effort=10.0 velocity=1.0 -> lower=0 upper=0.93 effort=50.0 velocity=1.0
- joint right_finger_joint: limit lower=-0.01 upper=0.94 effort=10.0 velocity=1.0 -> lower=-0.01 upper=0.94 effort=50.0 velocity=1.0
- joint right_inner_knuckle_joint: limit lower=-0.01 upper=0.94 effort=10.0 velocity=1.0 -> lower=-0.01 upper=0.94 effort=50.0 velocity=1.0
- joint right_outer_knuckle_joint: limit lower=-0.01 upper=0.94 effort=10.0 velocity=1.0 -> lower=-0.01 upper=0.94 effort=50.0 velocity=1.0
- joint shoulder_lift_joint: limit lower=-3.04 upper=3.04 effort=150 velocity=3.14159265359 -> lower=-3.04 upper=3.04 effort=150.0 velocity=50
- joint shoulder_pan_joint: limit lower=-3.04 upper=3.04 effort=150 velocity=3.14159265359 -> lower=-3.04 upper=3.04 effort=150.0 velocity=50
- joint wrist_1_joint: limit lower=-3.04 upper=3.04 effort=28 velocity=3.14159265359 -> lower=-3.04 upper=3.04 effort=28.0 velocity=50
- joint wrist_2_joint: limit lower=-3.04 upper=3.04 effort=28 velocity=3.14159265359 -> lower=-3.04 upper=3.04 effort=28.0 velocity=50
- joint wrist_3_joint: limit lower=-3.04 upper=3.04 effort=28 velocity=3.14159265359 -> lower=-3.04 upper=3.04 effort=28.0 velocity=50
